File: Asservissement_CDFR_2025/Asservissement_CDFR_2025.kicad_pcb (KiCad board)
At the start: 2 copper layers, 87 x 115 mm, 181 parts, among them IC1 A3930KJPTR-T, IC2 A3930KJPTR-T, J1 Connecteur batterie, J10 Free Connecteur, J13 Connecteur Odométrie, J2 Conn_01x03, J3 Conn_01x05, J4 Connecteur Programmation, J5 Conn_01x03, J6 Connecteur Odométrie, J7 Conn_01x03, J8 Conn_01x03, J9 Conn_01x05, Q1 QM6006D, Q10 QM6006D, Q11 QM6006D, Q12 QM6006D, Q13 Q_NMOS_GDS, Q2 QM6006D, Q3 QM6006D, Q4 QM6006D, Q5 QM6006D, Q6 QM6006D, Q7 QM6006D, Q8 QM6006D, Q9 QM6006D, SW1 SW_Push, SW2 SW_Push, SW3 SW_Push, U1 LM317_SOT-223, U3 STM32F401RCTx, U4 LMR16020PDDA

Commit message: lets go
Parts:
- removed C8: 470uF, Capacitor_SMD:CP_Elec_10x10.5
- removed H5, H6, H7, H8: MountingHole_Pad, MountingHole:MountingHole_2.7mm_Pad_Via
- removed J13: Connecteur Odométrie, Connector_JST:JST_XH_B4B-XH-A_1x04_P2.50mm_Vertical
- removed L2: 10uH, IHLP2525CZER100M01:IND_IHLP_2525_CZ-M
- removed TP27, TP28, TP29, TP30, TP31, TP32, TP33, TP34, TP35, TP36: TestPoint, TestPoint:TestPoint_Pad_D1.0mm
- removed U4: LMR16020PDDA, Package_SO:SOIC-8-1EP_3.9x4.9mm_P1.27mm_EP2.41x3.3mm
- removed kibuzzard-637D41F7: G***, kibuzzard-637D41F7
- removed kibuzzard-637D4204: G***, kibuzzard-637D4204
- removed kibuzzard-637D4217: G***, kibuzzard-637D4217
- removed kibuzzard-637D436E: G***, kibuzzard-637D436E
- removed kibuzzard-637D4374: G***, kibuzzard-637D4374
- removed kibuzzard-637D437D: G***, kibuzzard-637D437D
- removed kibuzzard-637D4386: G***, kibuzzard-637D4386
- removed kibuzzard-637D438C: G***, kibuzzard-637D438C
- removed kibuzzard-637D43BC: G***, kibuzzard-637D43BC
- removed kibuzzard-637D43CD: G***, kibuzzard-637D43CD
- removed kibuzzard-637D4446 (x2): G***, kibuzzard-637D4446
- removed kibuzzard-637D4455: G***, kibuzzard-637D4455
- removed kibuzzard-637D4463 (x2): G***, kibuzzard-637D4463
- removed kibuzzard-637D44C4: G***, kibuzzard-637D44C4
- removed kibuzzard-637D44E0: G***, kibuzzard-637D44E0
- removed kibuzzard-637D4536: G***, kibuzzard-637D4536
- removed kibuzzard-637D45A0: G***, kibuzzard-637D45A0
- removed kibuzzard-eD: G***, kibuzzard-637D447D
- added C14: 220uF, Capacitor_SMD:CP_Elec_10x10.5, F.Cu at (41.4, 73.5)
- added C15: 100uF, Capacitor_SMD:CP_Elec_10x10.5, F.Cu at (51.8, 97.5)
- added C34: 470nF, Capacitor_SMD:C_0805_2012Metric_Pad1.18x1.45mm_HandSolder, F.Cu at (84.7, 62.4)
- added C35: 1uF, Capacitor_SMD:C_0805_2012Metric_Pad1.18x1.45mm_HandSolder, F.Cu at (88.5, 62.4)
- added C36: 47nF, Capacitor_SMD:C_0805_2012Metric_Pad1.18x1.45mm_HandSolder, F.Cu at (92.6, 66.3)
- added C37: 47nF, Capacitor_SMD:C_0805_2012Metric_Pad1.18x1.45mm_HandSolder, F.Cu at (92.6, 70.1)
- added C38: 47nF, Capacitor_SMD:C_0805_2012Metric_Pad1.18x1.45mm_HandSolder, F.Cu at (92.6, 73.8)
- added C39: 1uF, Capacitor_SMD:C_0805_2012Metric_Pad1.18x1.45mm_HandSolder, F.Cu at (95.2, 77.0)
- added C40: 470uF, Capacitor_SMD:CP_Elec_10x10.5, F.Cu at (88.6, 55.5)
- added CT3: 470pF, Capacitor_SMD:C_0805_2012Metric_Pad1.18x1.45mm_HandSolder, F.Cu at (79.2, 79.7)
- added IC3: A3930KJPTR-T, A3930KJPTR-T:A3930KJPTRT, F.Cu at (84.7, 69.5)
- added J11: Conn_01x03, TerminalBlockBend:CUI_TBP02R1-381-03BE, B.Cu at (113.9, 54.6)
- added L1: 10uH, IHLP2525CZER100M01:IND_IHLP_2525_CZ-M, F.Cu at (41.6, 83.0)
- added Q14: QM6006D, Package_TO_SOT_SMD:TO-252-2, F.Cu at (116.8, 74.3)
- added Q15: QM6006D, Package_TO_SOT_SMD:TO-252-2, F.Cu at (116.8, 61.5)
- added Q16: QM6006D, Package_TO_SOT_SMD:TO-252-2, F.Cu at (109.8, 74.3)
- added Q17: QM6006D, Package_TO_SOT_SMD:TO-252-2, F.Cu at (109.8, 61.5)
- added Q18: QM6006D, Package_TO_SOT_SMD:TO-252-2, F.Cu at (102.8, 74.3)
- added Q19: QM6006D, Package_TO_SOT_SMD:TO-252-2, F.Cu at (102.8, 61.5)
- added R1: 56k, Resistor_SMD:R_0805_2012Metric_Pad1.20x1.40mm_HandSolder, F.Cu at (82.4, 126.2)
- added R46: 56k, Resistor_SMD:R_0805_2012Metric_Pad1.20x1.40mm_HandSolder, F.Cu at (71.8, 59.9)
- added R47: 390K, Resistor_SMD:R_0805_2012Metric_Pad1.20x1.40mm_HandSolder, F.Cu at (83.1, 79.7)
- added R48: 2.2k, Resistor_SMD:R_0805_2012Metric_Pad1.20x1.40mm_HandSolder, F.Cu at (85.0, 79.7)
- added R49: 4.7k, Resistor_SMD:R_0805_2012Metric_Pad1.20x1.40mm_HandSolder, F.Cu at (84.0, 82.5)
- added R50: 100k, Resistor_SMD:R_0805_2012Metric_Pad1.20x1.40mm_HandSolder, F.Cu at (86.9, 79.7)
- added R51: 47k, Resistor_SMD:R_0805_2012Metric_Pad1.20x1.40mm_HandSolder, F.Cu at (90.8, 79.6)
- added R52: 15k, Resistor_SMD:R_0805_2012Metric_Pad1.20x1.40mm_HandSolder, F.Cu at (88.9, 79.6)
- added R53: 560, Resistor_SMD:R_0805_2012Metric_Pad1.20x1.40mm_HandSolder, F.Cu at (96.4, 72.7)
- added R54: 560, Resistor_SMD:R_0805_2012Metric_Pad1.20x1.40mm_HandSolder, F.Cu at (96.4, 67.0)
- added R55: 0.018, Resistor_SMD:R_2512_6332Metric, F.Cu at (97.2, 57.9)
- added R56: 560, Resistor_SMD:R_0805_2012Metric_Pad1.20x1.40mm_HandSolder, F.Cu at (96.4, 70.8)
- added R57: 560, Resistor_SMD:R_0805_2012Metric_Pad1.20x1.40mm_HandSolder, F.Cu at (96.4, 65.0)
- added R58: 560, Resistor_SMD:R_0805_2012Metric_Pad1.20x1.40mm_HandSolder, F.Cu at (96.4, 68.8)
- added R59: 560, Resistor_SMD:R_0805_2012Metric_Pad1.20x1.40mm_HandSolder, F.Cu at (96.4, 63.1)
- added R8: 100k, Resistor_SMD:R_0805_2012Metric_Pad1.20x1.40mm_HandSolder, F.Cu at (72.3, 106.5)
- added RT3: 56k, Resistor_SMD:R_0805_2012Metric_Pad1.20x1.40mm_HandSolder, F.Cu at (81.2, 79.7)
- added TP15: TestPoint, TestPoint:TestPoint_Pad_D1.0mm, B.Cu at (-27.1, 69.8)
- added TP16: TestPoint, TestPoint:TestPoint_Pad_D1.0mm, B.Cu at (-27.1, 72.8)
- added TP17: TestPoint, TestPoint:TestPoint_Pad_D1.0mm, B.Cu at (-27.1, 75.8)
- added TP18: TestPoint, TestPoint:TestPoint_Pad_D1.0mm, B.Cu at (-27.1, 78.9)
- added TP19: TestPoint, TestPoint:TestPoint_Pad_D1.0mm, B.Cu at (-30.1, 69.8)
- added TP20: TestPoint, TestPoint:TestPoint_Pad_D1.0mm, B.Cu at (-30.1, 72.8)
- added TP21: TestPoint, TestPoint:TestPoint_Pad_D1.0mm, B.Cu at (-30.1, 75.8)
- added TP22: TestPoint, TestPoint:TestPoint_Pad_D1.0mm, B.Cu at (-30.1, 78.9)
- added TP23: TestPoint, TestPoint:TestPoint_Pad_D1.0mm, B.Cu at (-33.2, 69.8)
- added TP24: TestPoint, TestPoint:TestPoint_Pad_D1.0mm, B.Cu at (-33.2, 72.8)
- added U2: LM317_SOT-223, Package_TO_SOT_SMD:SOT-223-3_TabPin2, F.Cu at (42.2, 97.0)
- C1, C16: value 470nF -> 10uF
- C11: value 100uF -> 100nF; footprint Capacitor_SMD:CP_Elec_10x10.5 -> Capacitor_SMD:C_0805_2012Metric_Pad1.18x1.45mm_HandSolder
- C12, C23: value 47nF -> 1uF
- C13, C24: value 47nF -> 470uF; footprint Capacitor_SMD:C_0805_2012Metric_Pad1.18x1.45mm_HandSolder -> Capacitor_SMD:CP_Elec_10x10.5
- C17, C2: value 10uF -> 100nF
- C18, C3: value 100nF -> 470nF
- C20, C5: value 1uF -> 47nF
- C21, C6: value 470uF -> 47nF; footprint Capacitor_SMD:CP_Elec_10x10.5 -> Capacitor_SMD:C_0805_2012Metric_Pad1.18x1.45mm_HandSolder
- C32: value 100nF -> 10uF
- C33: value 220uF -> 100nF; footprint Capacitor_SMD:CP_Elec_10x10.5 -> Capacitor_SMD:C_0805_2012Metric_Pad1.18x1.45mm_HandSolder
- D1: value LED -> D_Zener; footprint LED_SMD:LED_0805_2012Metric_Pad1.15x1.40mm_HandSolder -> Diode_SMD:D_SOD-123
- D2: value LED -> D_Filled; footprint LED_SMD:LED_0805_2012Metric_Pad1.15x1.40mm_HandSolder -> B170B:DIOM505270X240
- D5: value D_Zener -> LED; footprint Diode_SMD:D_SOD-123 -> LED_SMD:LED_0805_2012Metric_Pad1.15x1.40mm_HandSolder
- D6: value DIODE -> LED; footprint B170B:DIOM505270X240 -> LED_SMD:LED_0805_2012Metric_Pad1.15x1.40mm_HandSolder
- J10: value Free Connecteur -> Conn_01x05; footprint Connector_PinHeader_2.54mm:PinHeader_1x08_P2.54mm_Vertical -> Connector_JST:JST_XH_B5B-XH-A_1x05_P2.50mm_Vertical
- J2, J8: value Conn_01x03 -> Conn_01x05; footprint TerminalBlockBend:CUI_TBP02R1-381-03BE -> Connector_JST:JST_XH_B5B-XH-A_1x05_P2.50mm_Vertical
- J3, J9: value Conn_01x05 -> Conn_01x03; footprint Connector_JST:JST_XH_B5B-XH-A_1x05_P2.50mm_Vertical -> TerminalBlockBend:CUI_TBP02R1-381-03BE; moved to B.Cu
- J6: value Connecteur Odométrie -> I2C_Master_Odo
- J7: value Conn_01x03 -> I2C_Slave
- Q13: value Q_NMOS_GDS -> QM6006D
- Q7: value QM6006D -> Q_NMOS_GDS
- R11: value 56k -> 47k
- R12: value 56k -> 15k
- R13, R42, R43: value 56k -> 560
- R15: value 560 -> 0.018; footprint Resistor_SMD:R_0805_2012Metric_Pad1.20x1.40mm_HandSolder -> Resistor_SMD:R_2512_6332Metric
- R17: value 0.018 -> 560; footprint Resistor_SMD:R_2512_6332Metric -> Resistor_SMD:R_0805_2012Metric_Pad1.20x1.40mm_HandSolder
- R18: value 390K -> 560
- R19: value 100k -> 560
- R2: value 2k4 -> 56k
- R23: value 560 -> 2k4
- R24: value 560 -> 3k9
- R25: value 560 -> 150
- R26: value 56k -> 4.7k
- R27: value 56k -> 2.2k
- R29, R30, R5, R6: value 560 -> 56k
- R3: value 150 -> 56k
- R31, R7: value 560 -> 390K
- R32: value 0.018 -> 2.2k; footprint Resistor_SMD:R_2512_6332Metric -> Resistor_SMD:R_0805_2012Metric_Pad1.20x1.40mm_HandSolder
- R33: value 390k -> 4.7k
- R34: value 4.7k -> 100k
- R37: value 4.7k -> 560
- R38: value 2.2k -> 560
- R39: value 2.2k -> 0.018; footprint Resistor_SMD:R_0805_2012Metric_Pad1.20x1.40mm_HandSolder -> Resistor_SMD:R_2512_6332Metric
- R4: value 3k9 -> 10k
- R40: value 47k -> 560
- R41: value 15k -> 560
- R44: value 10k -> 56k
- R45: value 100k -> 56k
- SW2: value SW_Push -> SW_Test
- SW3: value SW_Push -> SW_Reset
- TP13, TP14: moved to F.Cu
- U1: value LM317_SOT-223 -> LMR16020PDDA; footprint Package_TO_SOT_SMD:SOT-223-3_TabPin2 -> Package_SO:SOIC-8-1EP_3.9x4.9mm_P1.27mm_EP2.41x3.3mm
- moved R9 111.7 mm to (186.6, 54.2)
- moved H2 106.4 mm to (120.6, 52.0)
- moved TP25 103.2 mm to (-33.2, 75.8)
- moved TP26 103.1 mm to (-33.2, 78.9)
- moved H3 102.1 mm to (38.6, 133.6)
- moved J9 95.9 mm to (118.2, 126.4), turned to 90 degrees
- moved J6 95.4 mm to (-22.0, 115.0), turned to 0 degrees
- moved TP8 95.3 mm to (-21.0, 78.9)
- moved TP12 94.8 mm to (-24.0, 78.9)
- moved TP11 94.6 mm to (-24.0, 75.8)
- moved TP10 94.5 mm to (-24.0, 72.8)
- moved D5 94.5 mm to (186.6, 50.3), turned to 90 degrees
- moved TP9 94.3 mm to (-24.0, 69.8)
- moved SW1 89.8 mm to (62.6, 41.3), turned to 90 degrees
- moved TP6 89.2 mm to (-21.0, 72.8)
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Connections:
- net Info_erreur_1_1 renamed /Info_Err_1_A
- net Info_erreur_2_1 renamed /Info_Err_2_A
- net Info_vitesse_1 renamed /Info_Speed_A
- net direction_controle_1 renamed /Dir_A
- net disable_1 renamed /Disable_A
- net frein_1 renamed /Brakes_A
- net reset_1 renamed /Reset_A
- net speed_controle_1 renamed /Speed_A
- C1 pad 1: Net-(IC1-CP2) -> +BATT
- C1 pad 2: Net-(IC1-CP1) -> GND
- C11 pad 1: +3.3V -> Net-(U1-BOOT)
- C11 pad 2: GND -> Net-(D2-K)
- C12 pad 1: Net-(IC1-CB) -> +BATT
- C12 pad 2: Net-(IC1-SB) -> GND
- C13 pad 1: Net-(IC1-CC) -> +BATT
- C13 pad 2: Net-(IC1-SC) -> GND
- C16 pad 1: Net-(IC2-CP2) -> +BATT
- C16 pad 2: Net-(IC2-CP1) -> GND
- C18 pad 1: +BATT -> Net-(IC2-CP2)
- C18 pad 2: GND -> Net-(IC2-CP1)
- C20 pad 1: +BATT -> Net-(IC2-CA)
- C20 pad 2: GND -> Net-(IC2-SA)
- C21 pad 1: +BATT -> Net-(IC2-CB)
- C21 pad 2: GND -> Net-(IC2-SB)
- C22 pad 1: Net-(IC2-CA) -> Net-(IC2-CC)
- C22 pad 2: Net-(IC2-SA) -> Net-(IC2-SC)
- C23 pad 1: Net-(IC2-CB) -> +BATT
- C23 pad 2: Net-(IC2-SB) -> GND
- C24 pad 1: Net-(IC2-CC) -> +BATT
- C24 pad 2: Net-(IC2-SC) -> GND
- C3 pad 1: +BATT -> Net-(IC1-CP2)
- C3 pad 2: GND -> Net-(IC1-CP1)
- C32 pad 1: Net-(U4-BOOT) -> +BATT
- C32 pad 2: Net-(D6-A) -> GND
- C33 pad 1: +5V -> +BATT
- C5 pad 1: +BATT -> Net-(IC1-CA)
- C5 pad 2: GND -> Net-(IC1-SA)
- C6 pad 1: +BATT -> Net-(IC1-CB)
- C6 pad 2: GND -> Net-(IC1-SB)
- C9 pad 1: Net-(IC1-CA) -> Net-(IC1-CC)
- C9 pad 2: Net-(IC1-SA) -> Net-(IC1-SC)
- D1 pad 2: +3.3V -> GND
- D2 pad 2: +5V -> GND
- D5 pad 2: GND -> +5V
- D6 pad 1: GND -> Net-(D6-K)
- D6 pad 2: Net-(D6-A) -> +3.3V
- IC1 pad 15: MODE_1 -> /Mode_A
- IC1 pad 19: Info_Courant_1 -> Net-(IC1-CSOUT_)
- IC1 pad 39: action_fault_1 -> /Action_Fault_A
- IC1 pad 44: info_direction_1 -> /Info_Dir_A
- IC2 pad 14: speed_controle_2 -> /Speed_B
- IC2 pad 15: MODE_2 -> /Mode_B
- IC2 pad 19: Info_Courant_2 -> Net-(IC2-CSOUT_)
- IC2 pad 2: reset_2 -> /Reset_B
- IC2 pad 39: action_fault_2 -> /Action_Fault_B
- IC2 pad 44: info_direction_2 -> /Info_Dir_B
- IC2 pad 46: disable_2 -> /Disable_B
- IC2 pad 5: Info_erreur_1_2 -> /Info_Err_1_B
- IC2 pad 6: Info_erreur_2_2 -> /Info_Err_2_B
- IC2 pad 7: Info_vitesse_2 -> /Info_Speed_B
- IC2 pad 8: frein_2 -> /Brakes_B
- IC2 pad 9: direction_controle_2 -> /Dir_B
- J10 pad 1: Free1 -> GND
- J10 pad 2: Free2 -> Net-(IC3-H3_)
- J10 pad 3: Free3 -> Net-(IC3-H2_)
- J10 pad 4: Free4 -> Net-(IC3-H1_)
- J10 pad 5: Free5 -> +5V
- J2 pad 1: Net-(IC1-SC) -> GND
- J2 pad 2: Net-(IC1-SB) -> Net-(IC1-H3_)
- J2 pad 3: Net-(IC1-SA) -> Net-(IC1-H2_)
- J3 pad 1: GND -> Net-(IC1-SC)
- J3 pad 2: Net-(IC1-H3_) -> Net-(IC1-SB)
- J3 pad 3: Net-(IC1-H2_) -> Net-(IC1-SA)
- J6 pad 1: GND -> unconnected-(J6-Pin_1-Pad1)
- J6 pad 2: Net-(J6-Pin_2) -> unconnected-(J6-Pin_2-Pad2)
- J6 pad 3: Net-(J6-Pin_3) -> unconnected-(J6-Pin_3-Pad3)
- J6 pad 4: +5V -> unconnected-(J6-Pin_4-Pad4)
- J8 pad 1: Net-(IC2-SC) -> GND
- J8 pad 2: Net-(IC2-SB) -> Net-(IC2-H3_)
- J8 pad 3: Net-(IC2-SA) -> Net-(IC2-H2_)
- J9 pad 1: GND -> Net-(IC2-SC)
- J9 pad 2: Net-(IC2-H3_) -> Net-(IC2-SB)
- J9 pad 3: Net-(IC2-H2_) -> Net-(IC2-SA)
- Q10 pad 2: Net-(IC2-SC) -> +BATT
- Q10 pad 3: Net-(IC2-CSP_) -> Net-(IC2-SB)
- Q12 pad 2: Net-(IC2-SA) -> +BATT
- Q12 pad 3: Net-(IC2-CSP_) -> Net-(IC2-SA)
- Q13 pad 1: Net-(D5-K) -> Net-(Q13-G)
- Q13 pad 2: Net-(J1-Pin_2) -> Net-(IC2-SA)
- Q13 pad 3: GND -> Net-(IC2-CSP_)
- Q2 pad 2: +BATT -> Net-(IC1-SC)
- Q2 pad 3: Net-(IC1-SB) -> Net-(IC1-CSP_)
- Q3 pad 3: Net-(IC1-SA) -> Net-(IC1-SB)
- Q4 pad 2: Net-(IC1-SC) -> Net-(IC1-SB)
- Q5 pad 2: Net-(IC1-SB) -> +BATT
- Q5 pad 3: Net-(IC1-CSP_) -> Net-(IC1-SA)
- Q7 pad 1: Net-(Q7-G) -> Net-(D1-K)
- Q7 pad 2: +BATT -> Net-(J1-Pin_2)
- Q7 pad 3: Net-(IC2-SC) -> GND
- Q8 pad 3: Net-(IC2-SB) -> Net-(IC2-SC)
- Q9 pad 2: +BATT -> Net-(IC2-SC)
- Q9 pad 3: Net-(IC2-SA) -> Net-(IC2-CSP_)
- R11 pad 2: Net-(IC1-H1_) -> Net-(IC1-VDSTH_)
- R12 pad 1: +5V -> Net-(IC1-VDSTH_)
- R12 pad 2: Net-(IC1-H2_) -> GND
- R13 pad 1: +5V -> Net-(IC1-GHC)
- R13 pad 2: Net-(IC1-H3_) -> Net-(Q1-G)
- R14 pad 2: Net-(Q4-G) -> Net-(Q2-G)
- R15 pad 1: Net-(IC1-GLB) -> Net-(IC1-CSP_)
- R15 pad 2: Net-(Q5-G) -> GND
- R16 pad 1: Net-(IC1-GLA) -> Net-(IC1-GHB)
- R16 pad 2: Net-(Q6-G) -> Net-(Q3-G)
- R17 pad 1: Net-(IC1-CSP_) -> Net-(IC1-GLB)
- R17 pad 2: GND -> Net-(Q4-G)
- R18 pad 1: Net-(IC1-RDEAD_) -> Net-(IC1-GHA)
- R18 pad 2: GND -> Net-(Q5-G)
- R19 pad 1: Net-(IC1-REF_) -> Net-(IC1-GLA)
- R19 pad 2: +5V -> Net-(Q6-G)
- R2 pad 1: +3.3V -> +BATT
- R2 pad 2: Net-(U1-ADJ) -> Net-(D1-K)
- R23 pad 1: Net-(IC2-GHC) -> +3.3V
- R23 pad 2: Net-(Q7-G) -> Net-(U2-ADJ)
- R24 pad 1: Net-(IC2-GHB) -> Net-(U2-ADJ)
- R24 pad 2: Net-(Q8-G) -> GND
- R25 pad 1: Net-(IC2-GHA) -> Net-(D6-K)
- R25 pad 2: Net-(Q9-G) -> GND
- R26 pad 1: +5V -> /Current_Info_A
- R26 pad 2: Net-(IC2-H1_) -> GND
- R27 pad 1: +5V -> /Current_Info_A
- R27 pad 2: Net-(IC2-H2_) -> Net-(IC1-CSOUT_)
- R28 pad 2: Net-(IC2-H3_) -> Net-(IC2-H1_)
- R29 pad 1: Net-(IC2-GLC) -> +5V
- R29 pad 2: Net-(Q10-G) -> Net-(IC2-H2_)
- R3 pad 1: Net-(D1-K) -> +5V
- R3 pad 2: GND -> Net-(U1-FB)
- R30 pad 1: Net-(IC2-GLB) -> +5V
- R30 pad 2: Net-(Q11-G) -> Net-(IC2-H3_)
- R31 pad 1: Net-(IC2-GLA) -> Net-(IC2-RDEAD_)
- R31 pad 2: Net-(Q12-G) -> GND
- R32 pad 1: Net-(IC2-CSP_) -> /Current_Info_B
- R32 pad 2: GND -> Net-(IC2-CSOUT_)
- R33 pad 1: Net-(IC2-RDEAD_) -> /Current_Info_B
- R34 pad 1: Info_Courant_1_uc -> Net-(IC2-REF_)
- R34 pad 2: GND -> +5V
- R37 pad 1: Info_Courant_2_uc -> Net-(IC2-GHC)
- R37 pad 2: GND -> Net-(Q8-G)
- R38 pad 1: Info_Courant_1_uc -> Net-(IC2-GLC)
- R38 pad 2: Info_Courant_1 -> Net-(Q9-G)
- R39 pad 1: Info_Courant_2_uc -> Net-(IC2-CSP_)
- R39 pad 2: Info_Courant_2 -> GND
- R4 pad 1: Net-(U1-ADJ) -> Net-(U1-FB)
- R40 pad 1: +5V -> Net-(IC2-GHB)
- R40 pad 2: Net-(IC1-VDSTH_) -> Net-(Q10-G)
- R41 pad 1: Net-(IC1-VDSTH_) -> Net-(IC2-GLB)
- R41 pad 2: GND -> Net-(Q11-G)
- R42 pad 1: +BATT -> Net-(IC2-GHA)
- R42 pad 2: Net-(D5-K) -> Net-(Q12-G)
- R43 pad 1: +5V -> Net-(IC2-GLA)
- R43 pad 2: Net-(U4-FB) -> Net-(Q13-G)
- R44 pad 1: Net-(U4-FB) -> +5V
- R44 pad 2: GND -> Net-(IC3-H1_)
- R45 pad 1: Net-(IC2-REF_) -> +5V
- R45 pad 2: +5V -> Net-(IC3-H2_)
- R5 pad 1: Net-(IC1-GHC) -> +5V
- R5 pad 2: Net-(Q1-G) -> Net-(IC1-H2_)
- R6 pad 1: Net-(IC1-GHB) -> +5V
- R6 pad 2: Net-(Q2-G) -> Net-(IC1-H3_)
- R7 pad 1: Net-(IC1-GHA) -> Net-(IC1-RDEAD_)
- R7 pad 2: Net-(Q3-G) -> GND
- R9 pad 1: Net-(D2-K) -> Net-(D5-K)
- TP1 pad 1: Info_Courant_2_uc -> action_fault_2
- TP10 pad 1: reset_2 -> speed_controle_2
- TP11 pad 1: Info_erreur_1_2 -> MODE_2
- TP12 pad 1: Info_erreur_2_2 -> Info_Courant_2_uc
- TP2 pad 1: MODE_2 -> info_direction_2
- TP25 pad 1: action_fault_1 -> MODE_1
- TP26 pad 1: info_direction_1 -> Info_Courant_1_uc
- TP3 pad 1: direction_controle_2 -> disable_2
- TP4 pad 1: speed_controle_2 -> reset_2
- TP5 pad 1: Info_vitesse_2 -> Info_erreur_1_2
- TP6 pad 1: frein_2 -> Info_erreur_2_2
- TP7 pad 1: action_fault_2 -> Info_vitesse_2
- TP8 pad 1: info_direction_2 -> frein_2
- TP9 pad 1: disable_2 -> direction_controle_2
- U1 pad 1: Net-(U1-ADJ) -> Net-(U1-BOOT)
- U1 pad 2: +3.3V -> +BATT
- U1 pad 3: +5V -> +BATT
- U3 pad 10: Free7 -> unconnected-(U3-PC2-Pad10)
- U3 pad 11: Info_Courant_2_uc -> /Current_Info_B
- U3 pad 14: MODE_1 -> /Mode_A
- U3 pad 15: Info_Courant_1_uc -> /Current_Info_A
- U3 pad 2: Free2 -> unconnected-(U3-PC13-Pad2)
- U3 pad 28: info_direction_1 -> /Info_Dir_A
- U3 pad 29: action_fault_1 -> /Action_Fault_A
- U3 pad 3: Free3 -> unconnected-(U3-PC14-Pad3)
- U3 pad 33: MODE_2 -> /Mode_B
- U3 pad 34: speed_controle_2 -> /Speed_B
- U3 pad 35: direction_controle_2 -> /Dir_B
- U3 pad 36: frein_2 -> /Brakes_B
- U3 pad 37: Info_vitesse_2 -> /Info_Speed_B
- U3 pad 38: Info_erreur_2_2 -> /Info_Err_2_B
- U3 pad 39: Info_erreur_1_2 -> /Info_Err_1_B
- U3 pad 4: Free4 -> unconnected-(U3-PC15-Pad4)
- U3 pad 40: reset_2 -> /Reset_B
- U3 pad 41: disable_2 -> /Disable_B
- U3 pad 42: info_direction_2 -> /Info_Dir_B
- U3 pad 43: action_fault_2 -> /Action_Fault_B
- U3 pad 44: Free8 -> unconnected-(U3-PA11-Pad44)
- U3 pad 54: odometrie2 -> unconnected-(U3-PD2-Pad54)
- U3 pad 55: Net-(J13-Pin_3) -> unconnected-(U3-PB3-Pad55)
- U3 pad 56: Net-(J6-Pin_2) -> unconnected-(U3-PB4-Pad56)
- U3 pad 57: Net-(J6-Pin_3) -> unconnected-(U3-PB5-Pad57)
- U3 pad 62: Free1 -> unconnected-(U3-PB9-Pad62)
- U3 pad 8: Free5 -> unconnected-(U3-PC0-Pad8)
- U3 pad 9: Free6 -> unconnected-(U3-PC1-Pad9)
Routing:
- net GND: track 496.6 -> 164.5 mm, vias 20 -> 59
- net +3.3V: track 236.9 -> 59.8 mm, vias 2 -> 10
- net +5V: track 223.3 -> 378.6 mm, vias 7 -> 11
- net NRST: track 76.2 -> 1.70 mm, vias 3 -> 0
- net info_direction_2: track 74.0 -> 0.00 mm, vias 1 -> 0
- net MODE_1: track 73.4 -> 0.00 mm, vias 1 -> 0
- net Info_Courant_1_uc: track 69.8 -> 0.00 mm, vias 3 -> 0
- net disable_2: track 68.7 -> 0.00 mm, vias 1 -> 0
- net reset_2: track 59.4 -> 0.00 mm, vias 1 -> 0
- net Net-(U3-PC11): track 59.2 -> 0.00 mm, vias 1 -> 0
- net Info_erreur_1_2: track 56.1 -> 0.00 mm, vias 1 -> 0
- net action_fault_2: track 55.0 -> 0.00 mm, vias 2 -> 0
- net Net-(U3-PC12): track 53.3 -> 0.00 mm, vias 1 -> 0
- net Info_erreur_2_2: track 52.0 -> 0.00 mm, vias 1 -> 0
- net Net-(IC1-CSP_): track 95.3 -> 44.3 mm, vias 8 -> 13
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- added copper zone on In1.Cu, net (none)
- added copper zone on In2.Cu, net +3.3V
- added copper zone on In2.Cu, net +BATT
- added copper zone on In1.Cu, net GND
- added copper zone on In2.Cu, net Net-(IC1-CSP_)
- added copper zone on In2.Cu, net Net-(IC2-CSP_)
- added copper zone on In2.Cu, net Net-(IC3-CSP_)
Other:
- board size 87 x 115 mm -> 90 x 89.5 mm
- copper layers 2 -> 4
- board text removed: "3.3V"
- board text removed: "5V"
- board text removed: "GND"
- board text removed: "JLCJLCJLCJLC"
- board text removed: "action_err_1"
- board text removed: "action_err_2"
- board text removed: "bouton"
- board text removed: "courant_1"
- board text removed: "courant_2"
- board text removed: "direction_1"
- board text removed: "direction_2"
- board text removed: "disable_1"
- board text removed: "disable_2"
- board text removed: "encodeur_1"
- board text removed: "encodeur_2"
- board text removed: "erreur_1_1"
- board text removed: "erreur_1_2"
- board text removed: "erreur_2_1"
- board text removed: "erreur_2_2"
- board text removed: "frein_1"
- board text removed: "frein_2"
- board text removed: "info_direction_2"
- board text removed: "mode_1"
- board text removed: "mode_2"
- board text removed: "reset"
- board text removed: "reset_1"
- board text removed: "reset_2"
- board text removed: "test"
- board text removed: "vitesse_1"
- board text removed: "vitesse_2"

Commit message: updates
Parts:
- added TP27: TestPoint, TestPoint:TestPoint_Pad_D1.0mm, F.Cu at (171.7, 100.3)
- added TP28: TestPoint, TestPoint:TestPoint_Pad_D1.0mm, F.Cu at (171.7, 103.3)
- added TP29: TestPoint, TestPoint:TestPoint_Pad_D1.0mm, F.Cu at (171.7, 106.4)
- added TP30: TestPoint, TestPoint:TestPoint_Pad_D1.0mm, F.Cu at (174.8, 100.3)
- added TP31: TestPoint, TestPoint:TestPoint_Pad_D1.0mm, F.Cu at (174.8, 103.3)
- added TP32: TestPoint, TestPoint:TestPoint_Pad_D1.0mm, F.Cu at (174.8, 106.4)
- added TP33: TestPoint, TestPoint:TestPoint_Pad_D1.0mm, F.Cu at (177.8, 100.3)
- added TP34: TestPoint, TestPoint:TestPoint_Pad_D1.0mm, F.Cu at (177.8, 103.3)
- added TP35: TestPoint, TestPoint:TestPoint_Pad_D1.0mm, F.Cu at (177.8, 106.4)
- added TP36: TestPoint, TestPoint:TestPoint_Pad_D1.0mm, F.Cu at (180.8, 100.3)
- added TP37: TestPoint, TestPoint:TestPoint_Pad_D1.0mm, F.Cu at (180.8, 103.3)
- added TP38: TestPoint, TestPoint:TestPoint_Pad_D1.0mm, F.Cu at (180.8, 106.4)
- TP1, TP10, TP11, TP12, TP15, TP16, TP17, TP18, TP19, TP2, TP20, TP21, TP22, TP23, TP24, TP25, TP26, TP3, TP4, TP5, TP6, TP7, TP8, TP9: moved to F.Cu
- moved TP10 220.8 mm to (195.1, 100.3), turned to 0 degrees
- moved TP11 220.8 mm to (195.1, 103.3), turned to 0 degrees
- moved TP12 220.8 mm to (195.1, 106.4), turned to 0 degrees
- moved TP9 219.1 mm to (192.0, 106.4), turned to 0 degrees
- moved TP24 217.5 mm to (180.8, 111.5), turned to 0 degrees
- moved TP25 217.5 mm to (180.8, 114.5), turned to 0 degrees
- moved TP26 217.5 mm to (180.8, 117.5), turned to 0 degrees
- moved TP23 216.3 mm to (177.8, 117.5), turned to 0 degrees
- moved TP7 214.4 mm to (192.0, 100.3), turned to 0 degrees
- moved TP8 214.4 mm to (192.0, 103.3), turned to 0 degrees
- moved TP5 212.6 mm to (188.9, 103.3), turned to 0 degrees
- moved TP6 212.6 mm to (188.9, 106.4), turned to 0 degrees
- moved TP21 210.9 mm to (177.8, 111.5), turned to 0 degrees
- moved TP22 210.9 mm to (177.8, 114.5), turned to 0 degrees
- moved TP19 209.7 mm to (174.8, 114.5), turned to 0 degrees
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Connections:
- net /bldc_driverC/Current_Info renamed /Current_Info_C
- D3 pad 2: Net-(D3-A) -> unconnected-(D3-A-Pad2)
- D4 pad 2: Net-(D4-A) -> unconnected-(D4-A-Pad2)
- IC1 pad 15: /Mode_A -> /Mode_Drive
- IC1 pad 2: /Reset_A -> /Reset_Drive
- IC1 pad 46: /Disable_A -> /Disable_Drive
- IC2 pad 15: /Mode_B -> /Mode_Drive
- IC2 pad 2: /Reset_B -> /Reset_Drive
- IC2 pad 46: /Disable_B -> /Disable_Drive
- IC3 pad 14: /bldc_driverC/Speed_Control -> /Speed_C
- IC3 pad 15: /bldc_driverC/Mode -> /Mode_Drive
- IC3 pad 2: /bldc_driverC/Reset -> /Reset_Drive
- IC3 pad 39: /bldc_driverC/Action_Fault -> /Action_Fault_C
- IC3 pad 44: /bldc_driverC/Info_Dir -> /Info_Dir_C
- IC3 pad 46: /bldc_driverC/Disable -> /Disable_Drive
- IC3 pad 5: /bldc_driverC/Info_Err_1 -> /Info_Err_1_C
- IC3 pad 6: /bldc_driverC/Info_Err_2 -> /Info_Err_2_C
- IC3 pad 7: /bldc_driverC/Info_Speed -> /Info_Speed_C
- IC3 pad 8: /bldc_driverC/Brakes -> /Brakes_C
- IC3 pad 9: /bldc_driverC/Dir -> /Dir_C
- SW1 pad 2: Net-(U3-PC11) -> unconnected-(SW1-Pad2)
- SW2 pad 2: Net-(U3-PC12) -> unconnected-(SW2-Pad2)
- TP1 pad 1: action_fault_2 -> unconnected-(TP1-Pad1)
- TP10 pad 1: speed_controle_2 -> unconnected-(TP10-Pad1)
- TP11 pad 1: MODE_2 -> unconnected-(TP11-Pad1)
- TP12 pad 1: Info_Courant_2_uc -> unconnected-(TP12-Pad1)
- TP15 pad 1: action_fault_1 -> unconnected-(TP15-Pad1)
- TP16 pad 1: info_direction_1 -> unconnected-(TP16-Pad1)
- TP17 pad 1: disable_1 -> unconnected-(TP17-Pad1)
- TP18 pad 1: reset_1 -> unconnected-(TP18-Pad1)
- TP19 pad 1: Info_erreur_1_1 -> unconnected-(TP19-Pad1)
- TP2 pad 1: info_direction_2 -> unconnected-(TP2-Pad1)
- TP20 pad 1: Info_erreur_2_1 -> unconnected-(TP20-Pad1)
- TP21 pad 1: Info_vitesse_1 -> unconnected-(TP21-Pad1)
- TP22 pad 1: frein_1 -> unconnected-(TP22-Pad1)
- TP23 pad 1: direction_controle_1 -> unconnected-(TP23-Pad1)
- TP24 pad 1: speed_controle_1 -> unconnected-(TP24-Pad1)
- TP25 pad 1: MODE_1 -> unconnected-(TP25-Pad1)
- TP26 pad 1: Info_Courant_1_uc -> unconnected-(TP26-Pad1)
- TP3 pad 1: disable_2 -> unconnected-(TP3-Pad1)
- TP4 pad 1: reset_2 -> unconnected-(TP4-Pad1)
- TP5 pad 1: Info_erreur_1_2 -> unconnected-(TP5-Pad1)
- TP6 pad 1: Info_erreur_2_2 -> unconnected-(TP6-Pad1)
- TP7 pad 1: Info_vitesse_2 -> unconnected-(TP7-Pad1)
- TP8 pad 1: frein_2 -> unconnected-(TP8-Pad1)
- TP9 pad 1: direction_controle_2 -> unconnected-(TP9-Pad1)
- U3 pad 14: /Mode_A -> /Info_Speed_C
- U3 pad 25: /Reset_A -> unconnected-(U3-PC5-Pad25)
- U3 pad 27: /Disable_A -> /Speed_C
- U3 pad 33: /Mode_B -> /Disable_Drive
- U3 pad 40: /Reset_B -> /I2C3_SDA
- U3 pad 41: /Disable_B -> /I2C3_CLK
- U3 pad 44: unconnected-(U3-PA11-Pad44) -> /Mode_Drive
- U3 pad 45: Net-(D3-A) -> unconnected-(U3-PA12-Pad45)
- U3 pad 50: Net-(D4-A) -> /Reset_Drive
- U3 pad 51: unconnected-(U3-PC10-Pad51) -> /Speed_C
- U3 pad 52: Net-(U3-PC11) -> /Dir_C
- U3 pad 53: Net-(U3-PC12) -> /Brakes_C
- U3 pad 54: unconnected-(U3-PD2-Pad54) -> /Info_Err_2_C
- U3 pad 55: unconnected-(U3-PB3-Pad55) -> /Info_Err_1_C
- U3 pad 56: unconnected-(U3-PB4-Pad56) -> /Action_Fault_C
- U3 pad 57: unconnected-(U3-PB5-Pad57) -> /Info_Dir_C
Routing:
- net /Mode_Drive: track 0.00 -> 49.4 mm
- net /Disable_Drive: track 0.00 -> 36.6 mm, vias 0 -> 2
- net /Action_Fault_A: track 1.75 -> 35.9 mm, vias 1 -> 2
- net /Action_Fault_B: track 1.75 -> 32.9 mm, vias 1 -> 2
- net /Info_Dir_B: track 0.00 -> 30.8 mm, vias 0 -> 2
- net /Info_Dir_A: track 1.64 -> 31.7 mm, vias 1 -> 2
- net /Info_Err_1_B: track 0.00 -> 30.0 mm, vias 0 -> 2
- net /Info_Err_2_B: track 0.00 -> 27.6 mm, vias 0 -> 2
- net /Info_Err_1_A: track 2.95 -> 28.5 mm, vias 1 -> 2
- net /Info_Speed_B: track 0.00 -> 24.9 mm, vias 0 -> 2
- net /Brakes_B: track 0.00 -> 24.1 mm, vias 0 -> 2
- net /Info_Err_2_A: track 2.03 -> 25.5 mm, vias 1 -> 2
- net /Dir_B: track 0.00 -> 23.1 mm, vias 0 -> 2
- net /Reset_Drive: track 0.00 -> 22.2 mm, vias 0 -> 2
- net /Brakes_A: track 5.16 -> 23.8 mm, vias 1 -> 2
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- removed copper zone on In1.Cu, net (none)
Other:
- board size 90 x 89.5 mm -> 90 x 90 mm

Commit message: awesome
Parts:
- removed C7: 470uF, Capacitor_SMD:CP_Elec_10x10.5
- removed D1: D_Zener, Diode_SMD:D_SOD-123
- removed Q7: Q_NMOS_GDS, Package_TO_SOT_SMD:TO-252-2
- removed R2: 56k, Resistor_SMD:R_0805_2012Metric_Pad1.20x1.40mm_HandSolder
- removed TP10, TP16, TP19, TP2, TP20, TP21, TP22, TP23, TP24, TP28, TP31, TP32, TP33, TP34, TP35, TP36, TP5, TP6, TP7, TP8, TP9: TestPoint, TestPoint:TestPoint_Pad_D1.0mm
- added kibuzzard-680E921E: G***, kibuzzard-680E921E, F.Cu at (58.2, 134.2)
- added kibuzzard-680E922A: G***, kibuzzard-680E922A, F.Cu at (100.6, 51.1)
- added kibuzzard-680E9252: G***, kibuzzard-680E9252, F.Cu at (122.0, 112.8)
- added kibuzzard-680E9A25: G***, kibuzzard-680E9A25, F.Cu at (55.6, 92.5)
- added kibuzzard-680E9A3A: G***, kibuzzard-680E9A3A, F.Cu at (55.6, 94.5)
- added kibuzzard-680E9A44: G***, kibuzzard-680E9A44, F.Cu at (55.6, 96.5)
- added kibuzzard-680E9A53: G***, kibuzzard-680E9A53, F.Cu at (55.6, 90.5)
- added kibuzzard-680E9E15: G***, kibuzzard-680E9E15, F.Cu at (37.2, 84.8)
- J11, J3, J9: moved to F.Cu
- TP1, TP11, TP12, TP15, TP17, TP18, TP25, TP26, TP27, TP29, TP3, TP30, TP37, TP38, TP4: moved to B.Cu
- moved TP11 121.1 mm to (74.0, 100.5), turned to 180 degrees
- moved TP12 114.9 mm to (81.1, 121.2), turned to 180 degrees
- moved D5 113.9 mm to (72.9, 56.4), turned to 180 degrees
- moved TP4 112.3 mm to (76.8, 105.8), turned to 180 degrees
- moved R9 109.8 mm to (76.8, 56.4), turned to 0 degrees
- moved TP38 109.7 mm to (78.4, 67.2), turned to 180 degrees
- moved TP1 108.4 mm to (77.8, 108.0), turned to 180 degrees
- moved JP1 105.6 mm to (68.9, 81.3), turned to 90 degrees
- moved J7 105.1 mm to (58.9, 83.2), turned to 0 degrees
- moved TP3 104.7 mm to (82.0, 119.2), turned to 180 degrees
- moved TP30 104.3 mm to (75.9, 67.2), turned to 180 degrees
- moved kibuzzard-637D428D 104.0 mm to (71.4, 79.0), turned to 180 degrees
- moved TP29 102.7 mm to (77.7, 65.2), turned to 180 degrees
- moved D3 102.4 mm to (66.7, 96.0)
- moved R20 102.4 mm to (66.7, 92.0)
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Connections:
- J1 pad 1: +BATT -> Net-(J1-Pin_1)
- J1 pad 2: Net-(J1-Pin_2) -> GND
- J11 pad 1: Net-(IC3-SC) -> Net-(IC3-SA)
- J11 pad 3: Net-(IC3-SA) -> Net-(IC3-SC)
- J3 pad 1: Net-(IC1-SC) -> Net-(IC1-SA)
- J3 pad 3: Net-(IC1-SA) -> Net-(IC1-SC)
- J6 pad 1: unconnected-(J6-Pin_1-Pad1) -> /I2C3_CLK
- J6 pad 2: unconnected-(J6-Pin_2-Pad2) -> /I2C3_SDA
- J6 pad 3: unconnected-(J6-Pin_3-Pad3) -> +3.3V
- J6 pad 4: unconnected-(J6-Pin_4-Pad4) -> GND
- J9 pad 1: Net-(IC2-SC) -> Net-(IC2-SA)
- J9 pad 3: Net-(IC2-SA) -> Net-(IC2-SC)
- TP1 pad 1: unconnected-(TP1-Pad1) -> /Speed_A
- TP11 pad 1: unconnected-(TP11-Pad1) -> /Current_Info_A
- TP12 pad 1: unconnected-(TP12-Pad1) -> /Info_Speed_A
- TP15 pad 1: unconnected-(TP15-Pad1) -> /Speed_B
- TP17 pad 1: unconnected-(TP17-Pad1) -> /Brakes_B
- TP18 pad 1: unconnected-(TP18-Pad1) -> /Dir_B
- TP25 pad 1: unconnected-(TP25-Pad1) -> /Current_Info_B
- TP26 pad 1: unconnected-(TP26-Pad1) -> /Info_Speed_B
- TP27 pad 1: unconnected-(TP27-Pad1) -> /Speed_C
- TP29 pad 1: unconnected-(TP29-Pad1) -> /Brakes_C
- TP3 pad 1: unconnected-(TP3-Pad1) -> /Brakes_A
- TP30 pad 1: unconnected-(TP30-Pad1) -> /Dir_C
- TP37 pad 1: unconnected-(TP37-Pad1) -> /Current_Info_C
- TP38 pad 1: unconnected-(TP38-Pad1) -> /Info_Speed_C
- TP4 pad 1: unconnected-(TP4-Pad1) -> /Dir_A
- U3 pad 51: /Speed_C -> unconnected-(U3-PC10-Pad51)
- U3 pad 8: unconnected-(U3-PC0-Pad8) -> /Current_Info_C
Routing:
- net /Disable_Drive: track 36.6 -> 114.7 mm, vias 2 -> 5
- net /Reset_Drive: track 22.2 -> 97.6 mm, vias 2 -> 8
- net +5V: track 371.9 -> 301.6 mm, vias 10 -> 9
- net /Info_Speed_C: track 0.00 -> 41.0 mm, vias 0 -> 2
- net /Brakes_C: track 0.00 -> 30.5 mm, vias 0 -> 2
- net /Dir_C: track 0.00 -> 30.0 mm, vias 0 -> 2
- net /Action_Fault_C: track 1.75 -> 31.6 mm, vias 1 -> 2
- net /Info_Dir_C: track 0.00 -> 28.2 mm, vias 0 -> 2
- net /Speed_C: track 0.00 -> 26.7 mm, vias 0 -> 2
- net /Info_Err_2_C: track 0.00 -> 25.0 mm, vias 0 -> 2
- net /Current_Info_C: track 1.80 -> 25.5 mm, vias 0 -> 2
- net /Current_Info_B: track 1.80 -> 24.9 mm, vias 0 -> 2
- net /Info_Err_1_C: track 0.00 -> 21.9 mm, vias 0 -> 2
- net /Mode_Drive: track 49.4 -> 68.1 mm, vias 0 -> 2
- net +BATT: track 422.5 -> 409.4 mm
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Other:
- board text added: "CDFR 2025 Carte d'asservissement Omni Rev1 ROBOTRONIK - Ludovic Bouchard"
- board text removed: "Asservissement CDFR Robotronik Phelma"
- board text removed: "Version 2024/2025 (rev. 4)"

Commit message: Rev1 Candidate
Parts:
- removed kibuzzard-637D42B7: G***, kibuzzard-637D42B7
- removed kibuzzard-637D42C2: G***, kibuzzard-637D42C2
- removed kibuzzard-637D42CB: G***, kibuzzard-637D42CB
- removed kibuzzard-637D42F0: G***, kibuzzard-637D42F0
- removed kibuzzard-637D4301: G***, kibuzzard-637D4301
- removed kibuzzard-637D4322: G***, kibuzzard-637D4322
- removed kibuzzard-637D4331: G***, kibuzzard-637D4331
- removed kibuzzard-680E9A25: G***, kibuzzard-680E9A25
- removed kibuzzard-680E9A3A: G***, kibuzzard-680E9A3A
- removed kibuzzard-680E9A44: G***, kibuzzard-680E9A44
- removed kibuzzard-680E9A53: G***, kibuzzard-680E9A53
- added F1: 0154010.DR, FuseHolder:FUSE_0154004.DR, F.Cu at (65.2, 54.3)
- added kibuzzard-6810B1F2: G***, kibuzzard-6810B1F2, F.Cu at (56.4, 85.2)
- added kibuzzard-6810B296: G***, kibuzzard-6810B296, F.Cu at (68.0, 102.5)
- added kibuzzard-6810B2DF: G***, kibuzzard-6810B2DF, F.Cu at (61.5, 88.8)
- added kibuzzard-6810B2E9: G***, kibuzzard-6810B2E9, F.Cu at (61.3, 91.2)
- added kibuzzard-6810B2F1: G***, kibuzzard-6810B2F1, F.Cu at (61.7, 93.8)
- added kibuzzard-6810B2F8: G***, kibuzzard-6810B2F8, F.Cu at (61.3, 96.2)
- added kibuzzard-6810B307: G***, kibuzzard-6810B307, F.Cu at (59.2, 99.8)
- added kibuzzard-6810B314: G***, kibuzzard-6810B314, F.Cu at (61.6, 99.8)
- added kibuzzard-6810B3A9: G***, kibuzzard-6810B3A9, F.Cu at (52.2, 105.0)
- added kibuzzard-6810B3D0: G***, kibuzzard-6810B3D0, F.Cu at (55.7, 99.5)
- added kibuzzard-6810B3D6: G***, kibuzzard-6810B3D6, F.Cu at (53.3, 98.8)
- added kibuzzard-6810B3E4: G***, kibuzzard-6810B3E4, F.Cu at (50.8, 98.5)
- added kibuzzard-6810B3EB: G***, kibuzzard-6810B3EB, F.Cu at (48.2, 99.0)
- added kibuzzard-6810B459: G***, kibuzzard-6810B459, F.Cu at (50.6, 93.8)
- added kibuzzard-6810B45F: G***, kibuzzard-6810B45F, F.Cu at (50.8, 91.2)
- added kibuzzard-6810B467: G***, kibuzzard-6810B467, F.Cu at (50.8, 88.5)
- added kibuzzard-6810B4F3: G***, kibuzzard-6810B4F3, F.Cu at (66.4, 85.0)
- added kibuzzard-6810B9D4: G***, kibuzzard-6810B9D4, F.Cu at (62.4, 75.2)
- added kibuzzard-6810C26F: G***, kibuzzard-6810C26F, F.Cu at (71.6, 54.4)
- added kibuzzard-6810C528: G***, kibuzzard-6810C528, F.Cu at (36.6, 92.2)
- added kibuzzard-6810C533: G***, kibuzzard-6810C533, F.Cu at (36.6, 99.8)
- D3: value LED -> RED LED
- D4: value LED -> GREEN LED
- D5, D6: value LED -> BLUE LED
- moved C11 84.0 mm to (61.8, 70.2), turned to 180 degrees
- moved D2 79.3 mm to (52.5, 71.2)
- moved U1 78.2 mm to (60.2, 66.3), turned to 180 degrees
- moved L1 75.2 mm to (52.5, 65.2)
- moved J4 75.0 mm to (55.6, 102.5), turned to -90 degrees
- moved R4 74.8 mm to (62.0, 62.4), turned to 0 degrees
- moved R3 69.2 mm to (58.3, 62.4), turned to 0 degrees
- moved U2 67.3 mm to (57.2, 80.1)
- moved D6 67.3 mm to (59.0, 75.2)
- moved R23 67.3 mm to (51.6, 79.2)
- moved R24 67.3 mm to (51.6, 75.5)
- moved R25 67.3 mm to (55.2, 75.2)
- moved TP14 64.5 mm to (61.6, 85.0)
- moved C15 59.0 mm to (41.8, 73.0)
- moved C14 55.4 mm to (41.8, 62.0), turned to 180 degrees
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Connections:
- D3 pad 2: unconnected-(D3-A-Pad2) -> /RedLED
- D4 pad 2: unconnected-(D4-A-Pad2) -> /GreenLED
- SW1 pad 2: unconnected-(SW1-Pad2) -> /BttPush
- SW2 pad 2: unconnected-(SW2-Pad2) -> /BttTest
- U3 pad 3: unconnected-(U3-PC14-Pad3) -> /BttTest
- U3 pad 4: unconnected-(U3-PC15-Pad4) -> /BttPush
- U3 pad 61: unconnected-(U3-PB8-Pad61) -> /RedLED
- U3 pad 62: unconnected-(U3-PB9-Pad62) -> /GreenLED
Routing:
- net NRST: track 1.70 -> 70.6 mm, vias 0 -> 1
- net +5V: track 301.6 -> 346.1 mm, vias 9 -> 10
- net /BttPush: track 0.00 -> 42.7 mm
- net SWDIO: track 0.00 -> 40.2 mm, vias 0 -> 1
- net /BttTest: track 0.00 -> 40.0 mm
- net SWCLK: track 0.00 -> 36.5 mm, vias 0 -> 2
- net /I2C_CLK: track 0.00 -> 25.2 mm, vias 0 -> 1
- net /I2C_SDA: track 0.00 -> 25.0 mm, vias 0 -> 1
- net /TX: track 0.00 -> 16.1 mm
- net /RX: track 0.00 -> 15.7 mm
- net Net-(J1-Pin_1): track 0.00 -> 15.1 mm
- net /I2C3_CLK: track 5.90 -> 19.5 mm, vias 0 -> 1
- net Net-(JP1-C): track 0.00 -> 12.4 mm
- net +3.3V: track 55.5 -> 67.1 mm, vias 9 -> 11
- net /I2C3_SDA: track 8.06 -> 18.7 mm, vias 0 -> 1
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
Commit message: final
Parts:
- F1: value 0154010.DR -> 0154010.DR
