File: Asservissement_CDFR_2025/Asservissement_CDFR_2025.kicad_sch (KiCad schematic)
At the start: 152 parts, among them IC1 A3930KJPTR-T, IC2 A3930KJPTR-T, J1 Connecteur batterie, J10 Free Connecteur, J13 Connecteur Odométrie, J2 Conn_01x03, J3 Conn_01x05, J4 Connecteur Programmation, J5 Conn_01x03, J6 Connecteur Odométrie, J7 Conn_01x03, J8 Conn_01x03, J9 Conn_01x05, Q1 QM6006D, Q10 QM6006D, Q11 QM6006D, Q12 QM6006D, Q13 Q_NMOS_GDS, Q2 QM6006D, Q3 QM6006D, Q4 QM6006D, Q5 QM6006D, Q6 QM6006D, Q7 QM6006D, Q8 QM6006D, Q9 QM6006D, SW1 SW_Push, SW2 SW_Push, SW3 SW_Push, U1 LM317_SOT-223, U3 STM32F401RCTx, U4 LMR16020PDDA

Commit message: lets go
Parts:
- removed C1, C16: 470nF, Capacitor_SMD:C_0805_2012Metric_Pad1.18x1.45mm_HandSolder, symbol Device:C
- removed C11: 100uF, Capacitor_SMD:CP_Elec_10x10.5, symbol Device:C_Polarized
- removed C12, C13, C22, C23, C24, C9: 47nF, Capacitor_SMD:C_0805_2012Metric_Pad1.18x1.45mm_HandSolder, symbol Device:C_Small
- removed C17, C2: 10uF, Capacitor_SMD:C_0805_2012Metric_Pad1.18x1.45mm_HandSolder, symbol Device:C
- removed C18, C3, C32: 100nF, Capacitor_SMD:C_0805_2012Metric_Pad1.18x1.45mm_HandSolder, symbol Device:C
- removed C19, C20, C4, C5: 1uF, Capacitor_SMD:C_0805_2012Metric_Pad1.18x1.45mm_HandSolder, symbol Device:C
- removed C21, C6, C7, C8: 470uF, Capacitor_SMD:CP_Elec_10x10.5, symbol Device:C_Polarized
- removed C33: 220uF, Capacitor_SMD:CP_Elec_10x10.5, symbol Device:C_Polarized
- removed CT1, CT2: 470pF, Capacitor_SMD:C_0805_2012Metric_Pad1.18x1.45mm_HandSolder, symbol Device:C
- removed D1, D2: LED, LED_SMD:LED_0805_2012Metric_Pad1.15x1.40mm_HandSolder, symbol Device:LED
- removed D5: D_Zener, Diode_SMD:D_SOD-123, symbol Device:D_Zener
- removed D6: DIODE, B170B:DIOM505270X240, symbol pspice:DIODE
- removed H1, H2, H3, H4: MountingHole_Pad, MountingHole:MountingHole_3.2mm_M3_Pad_Via, symbol Mechanical:MountingHole_Pad
- removed H5, H6, H7, H8: MountingHole_Pad, MountingHole:MountingHole_2.7mm_Pad_Via, symbol Mechanical:MountingHole_Pad
- removed IC1, IC2: A3930KJPTR-T, A3930KJPTR-T:A3930KJPTRT, symbol a3930kjptr-t:A3930KJPTR-T
- removed J1: Connecteur batterie, TerminalBlockBend:CUI_TBP01R1-508-02BE, symbol Connector:Screw_Terminal_01x02
- removed J10: Free Connecteur, Connector_PinHeader_2.54mm:PinHeader_1x08_P2.54mm_Vertical, symbol Connector:Conn_01x08_Male
- removed J13: Connecteur Odométrie, Connector_JST:JST_XH_B4B-XH-A_1x04_P2.50mm_Vertical, symbol Connector_Generic:Conn_01x04
- removed J2, J8: Conn_01x03, TerminalBlockBend:CUI_TBP02R1-381-03BE, symbol Connector_Generic:Conn_01x03
- removed J3, J9: Conn_01x05, Connector_JST:JST_XH_B5B-XH-A_1x05_P2.50mm_Vertical, symbol Connector_Generic:Conn_01x05
- removed L2: 10uH, IHLP2525CZER100M01:IND_IHLP_2525_CZ-M, symbol Device:L
- removed Q1, Q10, Q11, Q12, Q2, Q3, Q4, Q5, Q6, Q7, Q8, Q9: QM6006D, Package_TO_SOT_SMD:TO-252-2, symbol Transistor_FET:QM6006D
- removed Q13: Q_NMOS_GDS, Package_TO_SOT_SMD:TO-252-2, symbol Device:Q_NMOS_GDS
- removed R11, R12, R13, R26, R27, R28, R42, R43, RT1, RT2: 56k, Resistor_SMD:R_0805_2012Metric_Pad1.20x1.40mm_HandSolder, symbol Device:R
- removed R14, R15, R16, R23, R24, R25, R29, R30, R31, R5, R6, R7: 560, Resistor_SMD:R_0805_2012Metric_Pad1.20x1.40mm_HandSolder, symbol Device:R
- removed R17, R32: 0.018, Resistor_SMD:R_2512_6332Metric, symbol Device:R
- removed R18: 390K, Resistor_SMD:R_0805_2012Metric_Pad1.20x1.40mm_HandSolder, symbol Device:R
- removed R19, R45: 100k, Resistor_SMD:R_0805_2012Metric_Pad1.20x1.40mm_HandSolder, symbol Device:R
- removed R2: 2k4, Resistor_SMD:R_0805_2012Metric_Pad1.20x1.40mm_HandSolder, symbol Device:R
- removed R3: 150, Resistor_SMD:R_0805_2012Metric_Pad1.20x1.40mm_HandSolder, symbol Device:R
- removed R33: 390k, Resistor_SMD:R_0805_2012Metric_Pad1.20x1.40mm_HandSolder, symbol Device:R
- removed R34, R37: 4.7k, Resistor_SMD:R_0805_2012Metric_Pad1.20x1.40mm_HandSolder, symbol Device:R
- removed R35, R40: 47k, Resistor_SMD:R_0805_2012Metric_Pad1.20x1.40mm_HandSolder, symbol Device:R
- removed R36, R41: 15k, Resistor_SMD:R_0805_2012Metric_Pad1.20x1.40mm_HandSolder, symbol Device:R
- removed R38, R39: 2.2k, Resistor_SMD:R_0805_2012Metric_Pad1.20x1.40mm_HandSolder, symbol Device:R
- removed R4: 3k9, Resistor_SMD:R_0805_2012Metric_Pad1.20x1.40mm_HandSolder, symbol Device:R
- removed R44: 10k, Resistor_SMD:R_0805_2012Metric_Pad1.20x1.40mm_HandSolder, symbol Device:R
- removed R9: 220, Resistor_SMD:R_0805_2012Metric_Pad1.20x1.40mm_HandSolder, symbol Device:R
- removed TP1, TP10, TP11, TP12, TP13, TP14, TP2, TP25, TP26, TP27, TP28, TP29, TP3, TP30, TP31, TP32, TP33, TP34, TP35, TP36, TP4, TP5, TP6, TP7, TP8, TP9: TestPoint, TestPoint:TestPoint_Pad_D1.0mm, symbol Connector:TestPoint
- removed U1: LM317_SOT-223, Package_TO_SOT_SMD:SOT-223-3_TabPin2, symbol Regulator_Linear:LM317_SOT-223
- removed U4: LMR16020PDDA, Package_SO:SOIC-8-1EP_3.9x4.9mm_P1.27mm_EP2.41x3.3mm, symbol LMR16020PDDA:LMR16020PDDA
- J6: value Connecteur Odométrie -> I2C_Master_Odo
- J7: value Conn_01x03 -> I2C_Slave
- SW2: value SW_Push -> SW_Test
- SW3: value SW_Push -> SW_Reset
Connections:
- net GND: no longer J6.1 (Pin_1)
- net at U3.56 (PB4): no longer J6.2 (Pin_2)
- net at U3.57 (PB5): no longer J6.3 (Pin_3)
- net +5V: no longer names the net of J6.4 (Pin_4)
- net Free1: no longer names the net of U3.62 (PB9)
- net Free2: no longer names the net of U3.2 (PC13)
- net Free3: no longer names the net of U3.3 (PC14)
- net Free4: no longer names the net of U3.4 (PC15)
- net Free5: no longer names the net of U3.8 (PC0)
- net Free6: no longer names the net of U3.9 (PC1)
- net Free7: no longer names the net of U3.10 (PC2)
- net Free8: no longer names the net of U3.44 (PA11)
- net Info_Courant_1_uc renamed Current_Info_A
- net Info_Courant_2_uc renamed Current_Info_B
- net Info_erreur_1_1 renamed Info_Err_1_A
- net Info_erreur_1_2 renamed Info_Err_1_B
- net Info_erreur_2_1 renamed Info_Err_2_A
- net Info_erreur_2_2 renamed Info_Err_2_B
- net Info_vitesse_1 renamed Info_Speed_A
- net Info_vitesse_2 renamed Info_Speed_B
- net MODE_1 renamed Mode_A
- net MODE_2 renamed Mode_B
- net action_fault_1 renamed Action_Fault_A
- net action_fault_2 renamed Action_Fault_B
- net direction_controle_1 renamed Dir_A
- net direction_controle_2 renamed Dir_B
- net disable_1 renamed Disable_A
- net disable_2 renamed Disable_B
- net frein_1 renamed Brakes_A
- net frein_2 renamed Brakes_B
- net info_direction_1 renamed Info_Dir_A
- net info_direction_2 renamed Info_Dir_B
- net odometrie2: no longer names the net of U3.54 (PD2)
- net reset_1 renamed Reset_A
- net reset_2 renamed Reset_B
- net speed_controle_1 renamed Speed_A
- net speed_controle_2 renamed Speed_B
- no-connect marks 15 -> 2
Other:
- added sheet Alim (alim.kicad_sch)
- added sheet Other (other.kicad_sch)
- added sheet bldc_driverA (bldc_driver.kicad_sch)
- added sheet bldc_driverB (bldc_driver.kicad_sch)
- added sheet bldc_driverC (bldc_driver.kicad_sch)
- note removed: "Alimentation"
- note removed: "Blank time 650ns"
- note removed: "CBOOT = QGATE × 20 / VBOOT Vboot = Vreg"
- note removed: "Cesf 20 times larger than the bootstrap capacitor"
- note removed: "ID max = 35A => Vds = 0.5V VDSTH = 0.5V"
- note removed: "ITRIP = (VREF - VOOS) / (RSENSE×AV) Av = 19 Voos = 0.32V Vref = 4V max (limité) Itrip = courant max"
- note removed: "Piste indépendant faible impédance pour lss"
- note removed: "Vdrain : close to the drain connections of the high-side FETs, with an independent trace"
- note removed: "tBLANK (µs) = 1260× CT (µF) fOSC ≈ 1/(RTCT + tBLANK + tDEAD) fOSC < fPWM"
- moved on the sheet: C10, C25, C26, C27, C28, C29, C30, C31, D3, D4, J4, J5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

Commit message: updates
Connections:
- net Disable_A is gone; now on net Speed_C: U3.27 (PB1)
- net Disable_B is gone; now on net I2C3_CLK: U3.41 (PA8)
- net Reset_B is gone; now on net I2C3_SDA: U3.40 (PC9)
- net +3.3V: now also J6.3 (Pin_3)
- net GND: now also J6.4 (Pin_4)
- net Mode_Drive: now reaches U3.44 (PA11)
- net at U3.45 (PA12): no longer D3.2 (A)
- net at D4.2 (A): no longer U3.50 (PA15)
- net Speed_C: now reaches U3.51 (PC10)
- net at SW1.2: no longer U3.52 (PC11)
- net at SW2.2: no longer U3.53 (PC12)
- net Info_Err_2_C: now reaches U3.54 (PD2)
- net Info_Err_1_C: now reaches U3.55 (PB3)
- net Action_Fault_C: now reaches U3.56 (PB4)
- net Info_Dir_C: now reaches U3.57 (PB5)
- net I2C3_CLK: now reaches J6.1 (Pin_1)
- net I2C3_SDA: now reaches J6.2 (Pin_2)
- net Mode_A renamed Info_Speed_C
- net Mode_B renamed Disable_Drive
- net Reset_A: no longer names the net of U3.25 (PC5)
- new net Brakes_C: U3.53 (PC12)
- new net Dir_C: U3.52 (PC11)
- new net Reset_Drive: U3.50 (PA15)
Other:
- note added: "PWM Speed_controle_A : TIM1_CH2N Speed_controle_B : TIM1_CH1N Speed_controle_C : TIM1_CH3N CONTEURS Info_vitesse_A : TIM2 Info_vitesse_B : TM3 Info_vitesse_C : TM4-5 ADC Info_Courant_A : ADC_IN1 Info_Courant_B : ADC_IN11 Info_Courant_C : ADC_INXX"
- note removed: "Speed_controle_1 : TIM1_CH2N Speed_controle_2 : TIM1_CH1N Info_vitesse_1 : TIM2 Info_vitesse_2 : TM3 Info_Courant_1 : ADC_IN1 Info_Courant_2 : ADC_IN11"
- moved on the sheet: D3, D4, J6, R20, R22, SW1, SW2

Commit message: awesome
Parts:
- J4, J5, J6, J7: now left out of the parts list
Connections:
- net Current_Info_C: now also U3.8 (PC0)
- net Speed_C: no longer U3.51 (PC10)
Other:
- note added: "Development/programming: Set BOOT0 high to enter bootloader mode, so you can flash new firmware if needed Normal use: Set BOOT0 low permanently after flashing your program."
- note added: "PWM Speed_controle_A : TIM1_CH2N Speed_controle_B : TIM1_CH1N Speed_controle_C : TIM1_CH3N CONTEURS Info_vitesse_A : TIM2 Info_vitesse_B : TM3 Info_vitesse_C : TM4-5 ADC Info_Courant_A : ADC_IN1 Info_Courant_B : ADC_IN11 Info_Courant_C : ADC_IN10"
- note removed: "PWM Speed_controle_A : TIM1_CH2N Speed_controle_B : TIM1_CH1N Speed_controle_C : TIM1_CH3N CONTEURS Info_vitesse_A : TIM2 Info_vitesse_B : TM3 Info_vitesse_C : TM4-5 ADC Info_Courant_A : ADC_IN1 Info_Courant_B : ADC_IN11 Info_Courant_C : ADC_INXX"
Changed lines of the file:
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@@
 	(wire
 		(pts
-			(xy 78.74 147.32) (xy 99.06 147.32)
+			(xy 76.2 147.32) (xy 99.06 147.32)
 		)
 		(stroke
@@
 	(wire
 		(pts
-			(xy 152.4 157.48) (xy 132.08 157.48)
+			(xy 153.67 157.48) (xy 132.08 157.48)
 		)
 		(stroke
@@
 	(wire
 		(pts
-			(xy 152.4 134.62) (xy 132.08 134.62)
+			(xy 154.94 134.62) (xy 132.08 134.62)
 		)
 		(stroke
@@
 	(wire
 		(pts
-			(xy 152.4 152.4) (xy 132.08 152.4)
+			(xy 153.67 152.4) (xy 132.08 152.4)
 		)
 		(stroke
@@
 	(wire
 		(pts
-			(xy 78.74 144.78) (xy 99.06 144.78)
-		)
-		(stroke
-			(width 0)
-			(type default)
-		)
-	)
-	(wire
-		(pts
 			(xy 85.09 83.82) (xy 59.69 83.82)
 		)
@@
 	(wire
 		(pts
-			(xy 152.4 78.74) (xy 132.08 78.74)
+			(xy 154.94 78.74) (xy 132.08 78.74)
 		)
 		(stroke
@@
 	(wire
 		(pts
-			(xy 78.74 134.62) (xy 99.06 134.62)
+			(xy 77.47 134.62) (xy 99.06 134.62)
 		)
 		(stroke
@@
 	(wire
 		(pts
-			(xy 78.74 137.16) (xy 99.06 137.16)
+			(xy 77.47 137.16) (xy 99.06 137.16)
 		)
 		(stroke
@@
 	(wire
 		(pts
-			(xy 78.74 139.7) (xy 99.06 139.7)
+			(xy 77.47 139.7) (xy 99.06 139.7)
 		)
 		(stroke
@@
 	(wire
 		(pts
-			(xy 152.4 104.14) (xy 132.08 104.14)
+			(xy 153.67 104.14) (xy 132.08 104.14)
 		)
 		(stroke
@@
 	(wire
 		(pts
-			(xy 152.4 132.08) (xy 132.08 132.08)
+			(xy 154.94 132.08) (xy 132.08 132.08)
 		)
 		(stroke
@@
 	(wire
 		(pts
-			(xy 152.4 129.54) (xy 132.08 129.54)
+			(xy 154.94 129.54) (xy 132.08 129.54)
 		)
 		(stroke
@@
 	(wire
 		(pts
-			(xy 78.74 149.86) (xy 99.06 149.86)
+			(xy 76.2 149.86) (xy 99.06 149.86)
 		)
 		(stroke
@@
 	(wire
 		(pts
-			(xy 152.4 101.6) (xy 132.08 101.6)
+			(xy 153.67 101.6) (xy 132.08 101.6)
 		)
 		(stroke
@@
 	(wire
 		(pts
-			(xy 78.74 127) (xy 99.06 127)
+			(xy 77.47 127) (xy 99.06 127)
 		)
 		(stroke
@@
 	(wire
 		(pts
-			(xy 152.4 154.94) (xy 132.08 154.94)
+			(xy 76.2 119.38) (xy 99.06 119.38)
 		)
 		(stroke
@@
 	(wire
 		(pts
-			(xy 119.38 57.15) (xy 127 57.15)
+			(xy 153.67 154.94) (xy 132.08 154.94)
 		)
 		(stroke
@@
 	(wire
 		(pts
-			(xy 116.84 49.53) (xy 116.84 57.15)
+			(xy 119.38 57.15) (xy 127 57.15)
 		)
 		(stroke
@@
 	(wire
 		(pts
-			(xy 165.1 116.84) (xy 132.08 116.84)
+			(xy 116.84 49.53) (xy 116.84 57.15)
 		)
 		(stroke
@@
 	(wire
 		(pts
-			(xy 111.76 73.66) (xy 111.76 71.12)
+			(xy 165.1 116.84) (xy 132.08 116.84)
 		)
 		(stroke
@@
 	(wire
 		(pts
-			(xy 200.66 46.99) (xy 218.44 46.99)
+			(xy 111.76 73.66) (xy 111.76 71.12)
 		)
 		(stroke
@@
 	(wire
 		(pts
-			(xy 114.3 162.56) (xy 114.3 166.37)
+			(xy 200.66 46.99) (xy 218.44 46.99)
 		)
 		(stroke
@@
 	(wire
 		(pts
-			(xy 43.18 147.32) (xy 43.18 149.86)
+			(xy 114.3 162.56) (xy 114.3 166.37)
 		)
 		(stroke
@@
 	(wire
 		(pts
-			(xy 152.4 124.46) (xy 132.08 124.46)
+			(xy 154.94 124.46) (xy 132.08 124.46)
 		)
 		(stroke
@@
 		)
 	)
-	(text "PWM\nSpeed_controle_A : TIM1_CH2N\nSpeed_controle_B : TIM1_CH1N\nSpeed_controle_C : TIM1_CH3N\n\nCONTEURS\nInfo_vitesse_A : TIM2\nInfo_vitesse_B : TM3\nInfo_vitesse_C : TM4-5\n\nADC\nInfo_Courant_A : ADC_IN1\nInfo_Courant_B : ADC_IN11\nInfo_Courant_C : ADC_INXX\n"
+	(text "PWM\nSpeed_controle_A : TIM1_CH2N\nSpeed_controle_B : TIM1_CH1N\nSpeed_controle_C : TIM1_CH3N\n\nCONTEURS\nInfo_vitesse_A : TIM2\nInfo_vitesse_B : TM3\nInfo_vitesse_C : TM4-5\n\nADC\nInfo_Courant_A : ADC_IN1\nInfo_Courant_B : ADC_IN11\nInfo_Courant_C : ADC_IN10\n"
 		(exclude_from_sim no)
-		(at 84.074 195.834 0)
+		(at 129.032 192.024 0)
 		(effects
 			(font
@@
 		)
 	)
+	(text "Development/programming: Set BOOT0 high to enter bootloader mode, \nso you can flash new firmware if needed\nNormal use: Set BOOT0 low permanently after flashing your program."
+		(exclude_from_sim no)
+		(at 13.462 107.95 0)
+		(effects
+			(font
+				(size 1.27 1.27)
+			)
+			(justify left)
+		)
+	)
 	(text "3,6 v max pour VBATT (alim pour quartz) et 4 pour VDD"
 		(exclude_from_sim no)
@@
 	)
 	(label "Brakes_B"
-		(at 152.4 157.48 180)
+		(at 153.67 157.48 180)
 		(effects
 			(font
@@
 		)
 	)
-	(label "Speed_C"
-		(at 78.74 144.78 0)
-		(effects
-			(font
-				(size 1.27 1.27)
-			)
-			(justify left bottom)
-		)
-	)
 	(label "Action_Fault_A"
 		(at 152.4 147.32 180)
@@
 	)
 	(label "Info_Err_1_C"
-		(at 152.4 129.54 180)
+		(at 154.94 129.54 180)
 		(effects
 			(font
@@
 	)
 	(label "Info_Dir_C"
-		(at 152.4 134.62 180)
+		(at 154.94 134.62 180)
 		(effects
 			(font
@@
 	)
 	(label "Info_Err_1_B"
-		(at 78.74 139.7 0)
+		(at 77.47 139.7 0)
 		(effects
 			(font
@@
 		)
 	)
-	(label "Current_Info_C"
-		(at 146.05 143.51 0)
-		(effects
-			(font
-				(size 1.27 1.27)
-			)
-			(justify left bottom)
-		)
-	)
 	(label "SWDIO"
 		(at 152.4 111.76 180)
@@
 	)
 	(label "Action_Fault_B"
-		(at 152.4 104.14 180)
+		(at 153.67 104.14 180)
 		(effects
 			(font
@@
 	)
 	(label "Info_Speed_C"
-		(at 152.4 78.74 180)
+		(at 154.94 78.74 180)
 		(effects
 			(font
@@
 	)
 	(label "Action_Fault_C"
-		(at 152.4 132.08 180)
+		(at 154.94 132.08 180)
 		(effects
 			(font
@@
 	)
 	(label "Speed_C"
-		(at 152.4 124.46 180)
+		(at 154.94 124.46 180)
 		(effects
 			(font
@@
 	)
 	(label "Info_Err_2_B"
-		(at 78.74 137.16 0)
+		(at 77.47 137.16 0)
 		(effects
 			(font
@@
 	)
 	(label "Current_Info_B"
-		(at 78.74 127 0)
+		(at 77.47 127 0)
 		(effects
 			(font
@@
 		)
 	)
+	(label "Current_Info_C"
+		(at 76.2 119.38 0)
+		(effects
+			(font
+				(size 1.27 1.27)
+			)
+			(justify left bottom)
+		)
+	)
 	(label "Speed_B"
-		(at 152.4 152.4 180)
+		(at 153.67 152.4 180)
 		(effects
 			(font
@@
 	)
 	(label "Brakes_C"
-		(at 78.74 149.86 0)
+		(at 76.2 149.86 0)
 		(effects
 			(font
@@
 	)
 	(label "Info_Speed_B"
-		(at 78.74 134.62 0)
+		(at 77.47 134.62 0)
 		(effects
 			(font
@@
 	)
 	(label "Dir_B"
-		(at 152.4 154.94 180)
+		(at 153.67 154.94 180)
 		(effects
 			(font
@@
 	)
 	(label "Dir_C"
-		(at 78.74 147.32 0)
+		(at 76.2 147.32 0)
 		(effects
 			(font
@@
 	)
 	(label "Info_Dir_B"
-		(at 152.4 101.6 180)
+		(at 153.67 101.6 180)
 		(effects
 			(font
@@
 		(unit 1)
 		(exclude_from_sim no)
-		(in_bom yes)
+		(in_bom no)
 		(on_board yes)
 		(dnp no)
@@
 		(unit 1)
 		(exclude_from_sim no)
-		(in_bom yes)
+		(in_bom no)
 		(on_board yes)
 		(dnp no)
@@
 		(unit 1)
 		(exclude_from_sim no)
-		(in_bom yes)
+		(in_bom no)
 		(on_board yes)
 		(dnp no)
@@
 		(unit 1)
 		(exclude_from_sim no)
-		(in_bom yes)
+		(in_bom no)
 		(on_board yes)
 		(dnp no)

Commit message: Rev1 Candidate
Parts:
- D3: value LED -> RED LED
- D4: value LED -> GREEN LED
- JP1, SW1, SW2, SW3: now left out of the parts list
Connections:
- net BttTest: now reaches U3.3 (PC14)
- net BttTest: now also SW2.2
- net BttPush: now reaches U3.4 (PC15)
- net BttPush: now also SW1.2
- net RedLED: now reaches U3.61 (PB8)
- net RedLED: now also D3.2 (A)
- net GreenLED: now reaches U3.62 (PB9)
- net GreenLED: now also D4.2 (A)
- no-connect marks 2 -> 8
Other:
- moved on the sheet: D3, D4, R20, R22, SW1, SW2

Commit message: final
Parts:
- J6, J7, SW1, SW2, SW3: now in the parts list

Commit message: tiny
Connections:
- net Action_Fault_A renamed ESF_A
- net Action_Fault_B renamed ESF_B
- net Action_Fault_C renamed ESF_C
Other:
- sheet bldc_driverA ports: added ESF; removed Action_Fault
- sheet bldc_driverB ports: added ESF; removed Action_Fault
- sheet bldc_driverC ports: added ESF; removed Action_Fault
