File: Asservissement_CDFR_2025/bldc_driver.kicad_sch (KiCad schematic)
At the start: 48 parts, among them IC1 A3930KJPTR-T, J2 Conn_01x05, J3 Conn_01x03, Q1 QM6006D, Q2 QM6006D, Q3 QM6006D, Q4 QM6006D, Q5 QM6006D, Q6 QM6006D

Commit message: updates
Parts:
- IC3: renamed from IC1; Mouser Part Number (none) -> C459252
- J10: renamed from J2; now left out of the parts list
- renumbered C1 to C32, C2 to C33, C3 to C34, C4 to C35, C5 to C36, C6 to C37, C9 to C38, C12 to C39, C13 to C40, CT1 to CT3, J3 to J11, Q1 to Q14, Q2 to Q15, Q3 to Q16, Q4 to Q17, Q5 to Q18, Q6 to Q19, R1 to R44, R5 to R45, R6 to R46, R7 to R47, R27 to R48, R26 to R49, R8 to R50, R11 to R51, R12 to R52, R13 to R53, R14 to R54, R15 to R55, R16 to R56, R17 to R57, R18 to R58, R19 to R59, RT1 to RT3, TP1 to TP27, TP2 to TP28, TP3 to TP29, TP4 to TP30, TP5 to TP31, TP6 to TP32, TP7 to TP33, TP8 to TP34, TP9 to TP35, TP10 to TP36, TP11 to TP37, TP12 to TP38
Connections:
- net Brakes: now also TP29.1
- net Current_Info: now also TP37.1
- net Dir: now also TP30.1
- net Info_Speed: now also TP38.1
- net Mode: now also TP28.1
- net Speed_Control: now also TP27.1

Commit message: awesome
Parts:
- removed TP28, TP31, TP32, TP33, TP34, TP35, TP36: TestPoint, TestPoint:TestPoint_Pad_D1.0mm, symbol Connector:TestPoint
- J11, TP27, TP29, TP30, TP37, TP38: now left out of the parts list
Connections:
- net at C36.2, IC3.31 (SA), Q18.3 (S)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: now also J11.1 (Pin_1); no longer J11.3 (Pin_3)
- net at C38.2, IC3.25 (SC), Q14.3 (S)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: now also J11.3 (Pin_3); no longer J11.1 (Pin_1)

Commit message: final
Parts:
- J10, J11: now in the parts list
Changed lines of the file:
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@@
 		(shape input)
 		(at 267.97 130.81 180)
-		(fields_autoplaced yes)
 		(effects
 			(font
@@
 		(shape output)
 		(at 71.12 91.44 180)
-		(fields_autoplaced yes)
 		(effects
 			(font
@@
 		(shape output)
 		(at 71.12 86.36 180)
-		(fields_autoplaced yes)
 		(effects
 			(font
@@
 		(shape input)
 		(at 267.97 135.89 180)
-		(fields_autoplaced yes)
 		(effects
 			(font
@@
 		(shape output)
 		(at 71.12 88.9 180)
-		(fields_autoplaced yes)
 		(effects
 			(font
@@
 		(shape output)
 		(at 267.97 148.59 180)
-		(fields_autoplaced yes)
 		(effects
 			(font
@@
 		(shape input)
 		(at 71.12 93.98 180)
-		(fields_autoplaced yes)
 		(effects
 			(font
@@
 		(shape input)
 		(at 101.6 58.42 90)
-		(fields_autoplaced yes)
 		(effects
 			(font
@@
 		(shape input)
 		(at 267.97 133.35 180)
-		(fields_autoplaced yes)
 		(effects
 			(font
@@
 		(shape output)
 		(at 267.97 146.05 180)
-		(fields_autoplaced yes)
 		(effects
 			(font
@@
 		(shape input)
 		(at 71.12 96.52 180)
-		(fields_autoplaced yes)
 		(effects
 			(font
@@
 		(shape output)
 		(at 119.38 58.42 90)
-		(fields_autoplaced yes)
 		(effects
 			(font
@@
 		(shape input)
 		(at 71.12 78.74 180)
-		(fields_autoplaced yes)
 		(effects
 			(font
@@
 		(shape output)
 		(at 104.14 182.88 180)
-		(fields_autoplaced yes)
 		(effects
 			(font
@@
 		(shape input)
 		(at 96.52 129.54 270)
-		(fields_autoplaced yes)
 		(effects
 			(font
@@
 		(shape input)
 		(at 99.06 129.54 270)
-		(fields_autoplaced yes)
 		(effects
 			(font
@@
 		(shape output)
 		(at 106.68 58.42 90)
-		(fields_autoplaced yes)
 		(effects
 			(font
@@
 		(unit 1)
 		(exclude_from_sim no)
-		(in_bom no)
+		(in_bom yes)
 		(on_board yes)
 		(dnp no)
@@
 		(unit 1)
 		(exclude_from_sim no)
-		(in_bom no)
+		(in_bom yes)
 		(on_board yes)
 		(dnp no)

Commit message: tiny
Connections:
- net Action_Fault renamed ESF
Changed lines of the file:
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@@
 		(shape input)
 		(at 267.97 130.81 180)
+		(fields_autoplaced yes)
 		(effects
 			(font
@@
 		(shape output)
 		(at 71.12 91.44 180)
+		(fields_autoplaced yes)
 		(effects
 			(font
@@
 		(shape output)
 		(at 71.12 86.36 180)
+		(fields_autoplaced yes)
 		(effects
 			(font
@@
 		(shape input)
 		(at 267.97 135.89 180)
+		(fields_autoplaced yes)
 		(effects
 			(font
@@
 		(shape output)
 		(at 71.12 88.9 180)
+		(fields_autoplaced yes)
 		(effects
 			(font
@@
 		(shape output)
 		(at 267.97 148.59 180)
+		(fields_autoplaced yes)
 		(effects
 			(font
@@
 		(shape input)
 		(at 71.12 93.98 180)
+		(fields_autoplaced yes)
 		(effects
 			(font
@@
 		(shape input)
 		(at 101.6 58.42 90)
+		(fields_autoplaced yes)
 		(effects
 			(font
@@
 		(shape input)
 		(at 267.97 133.35 180)
+		(fields_autoplaced yes)
 		(effects
 			(font
@@
 		(shape output)
 		(at 267.97 146.05 180)
+		(fields_autoplaced yes)
 		(effects
 			(font
@@
 		(shape input)
 		(at 71.12 96.52 180)
+		(fields_autoplaced yes)
 		(effects
 			(font
@@
 		)
 	)
-	(hierarchical_label "Action_Fault"
-		(shape output)
+	(hierarchical_label "ESF"
+		(shape input)
 		(at 119.38 58.42 90)
+		(fields_autoplaced yes)
 		(effects
 			(font
@@
 		(shape input)
 		(at 71.12 78.74 180)
+		(fields_autoplaced yes)
 		(effects
 			(font
@@
 		(shape output)
 		(at 104.14 182.88 180)
+		(fields_autoplaced yes)
 		(effects
 			(font
@@
 		(shape input)
 		(at 96.52 129.54 270)
+		(fields_autoplaced yes)
 		(effects
 			(font
@@
 		(shape input)
 		(at 99.06 129.54 270)
+		(fields_autoplaced yes)
 		(effects
 			(font
@@
 		(shape output)
 		(at 106.68 58.42 90)
+		(fields_autoplaced yes)
 		(effects
 			(font

Commit message: updates
Parts:
- C36, C37, C38: value 47nF -> 220nF
- Q14, Q15, Q16, Q17, Q18, Q19: value QM6006D -> FQD50N06
- R47: value 390K -> 37k; Field4 960 ns -> 900ns Deadtime
- R53, R54, R56, R57, R58, R59: value 560 -> 10
Other:
- note added: "10"
- note added: "15 kΩ 220 pF"
- note added: "220nF"
- note added: "37k"
- note added: "FQD50N06"
- moved on the sheet: C32, C33, C34, C35, CT3, J10, J11, R47, R48, R49, R51, R52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

Commit message: updates
Other:
- note removed: "10"
- note removed: "220nF"
Changed lines of the file:
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@@
 		)
 	)
-	(text "220nF"
-		(exclude_from_sim no)
-		(at 136.398 108.712 0)
+	(text "37k"
+		(exclude_from_sim no)
+		(at 105.156 159.766 0)
 		(effects
 			(font
@@
 		)
 	)
-	(text "37k"
-		(exclude_from_sim no)
-		(at 105.156 159.766 0)
+	(text "15 kΩ 220 pF"
+		(exclude_from_sim no)
+		(at 79.756 152.146 0)
 		(effects
 			(font
@@
 		)
 	)
-	(text "15 kΩ 220 pF"
-		(exclude_from_sim no)
-		(at 79.756 152.146 0)
-		(effects
-			(font
-				(size 3 3)
-				(thickness 0.6)
-				(bold yes)
-				(color 255 12 6 1)
-			)
-		)
-	)
-	(text "10"
-		(exclude_from_sim no)
-		(at 154.94 118.11 0)
-		(effects
-			(font
-				(size 3 3)
-				(thickness 0.6)
-				(bold yes)
-				(color 255 12 6 1)
-			)
-		)
-	)
 	(text "Cesf 20 times larger \nthan the bootstrap capacitor"
 		(exclude_from_sim no)
@@
 		)
 		(property "Value" "TestPoint"
-			(at 273.05 149.8599 90)
+			(at 273.05 148.5899 90)
 			(effects
 				(font
@@
 		(on_board yes)
 		(dnp no)
-		(fields_autoplaced yes)
 		(property "Reference" "TP37"
 			(at 273.05 144.7799 90)
+			(show_name yes)
 			(effects
 				(font
@@
 		)
 		(property "Value" "TestPoint"
-			(at 273.05 147.3199 90)
-			(effects
-				(font
+			(at 273.05 146.0499 90)
+			(effects
+				(font
